File: NUsense/Power.sch (KiCad schematic (older format))
At the start: 13 parts

Commit message: Correct broken files
Parts:
- added C?: 0.1uF, symbol C
- added C?: 1uF, symbol C
- added C?: 47uF, symbol C
- added C?: 100nF, symbol C
- added C?: 10uF, symbol C
- added D? (x2): D_Schottky, symbol D_Schottky
- added Q?: Q_PMOS_GDS, symbol Q_PMOS_GDS
- added Q?: 2N2219, TO_SOT_Packages_THT:TO-39-3, symbol 2N2219
- added R? (x2): 47K, symbol R
- added U?: LD1086D2M33, symbol LD1086D2M33
- C?: value CP1 -> 68uF
- R? (x4): value R -> 100K
- R?: value R -> 22K
Connections:
- net labels added: +3.3V, +5V, DXL_PWR, DXL_PWR_EN
- wire segments 40 -> 70
