File: NUsense/RS485.sch (KiCad schematic (older format))
At the start: 15 parts, among them J18? MOLEX22-03-5045, U21? MAX3443ECSA+

Commit message: Correct broken files
Parts:
- removed C? (x2): C, symbol C
- removed D? (x2): D_Schottky, symbol D_Schottky
- removed Q?: Q_PMOS_GDS, symbol Q_PMOS_GDS
- removed Q?: 2N2219, TO_SOT_Packages_THT:TO-39-3, symbol 2N2219
- removed R? (x2): R, symbol R
- C? (x2): value C -> 0.1uF
- R? (x2): value R -> 10
Connections:
- net DXL_485+_1 renamed DXL_485+
- net DXL_485-_1 renamed DXL_485-
- net DXL_DIR_1 renamed DXL_DIR
- net DXL_RXD_1 renamed DXL_RXD
- net DXL_TXD_1 renamed DXL_TXD
- net VDD5o0V renamed +5V
Changed lines of the file:
@@
 LIBS:valves
 LIBS:ADM6713RAKS
+LIBS:Header_Connectors
 LIBS:MPU6000
 LIBS:NUbots
 LIBS:STM32F746ZGT6
-LIBS:Header_Connectors
 LIBS:NUsense-cache
 EELAYER 25 0
@@
 	1    0    0    -1
 $EndComp
-Text GLabel 3750 2550 1    60   Input ~ 0
-VDD5o0V
 $Comp
 L R R?
@@
 P 5800 3750
 F 0 "C?" H 5825 3850 50  0000 L CNN
-F 1 "C" H 5825 3650 50  0000 L CNN
+F 1 "0.1uF" H 5825 3650 50  0000 L CNN
 F 2 "" H 5838 3600 50  0001 C CNN
 F 3 "" H 5800 3750 50  0001 C CNN
@@
 	1    0    0    -1
 $EndComp
-Text GLabel 6100 3500 2    60   Input ~ 0
-VDD5o0V
 $Comp
 L R R?
@@
 P 6700 3300
 F 0 "R?" V 6780 3300 50  0000 C CNN
-F 1 "R" V 6700 3300 50  0000 C CNN
+F 1 "10" V 6700 3300 50  0000 C CNN
 F 2 "" V 6630 3300 50  0001 C CNN
 F 3 "" H 6700 3300 50  0001 C CNN
@@
 P 6700 3200
 F 0 "R?" V 6780 3200 50  0000 C CNN
-F 1 "R" V 6700 3200 50  0000 C CNN
+F 1 "10" V 6700 3200 50  0000 C CNN
 F 2 "" V 6630 3200 50  0001 C CNN
 F 3 "" H 6700 3200 50  0001 C CNN
@@
 	0    -1   -1   0
 $EndComp
-Text GLabel 3550 3600 0    60   Input ~ 0
-DXL_DIR_1
-Text GLabel 3550 3500 0    60   Input ~ 0
-DXL_TXD_1
-Text GLabel 3550 3200 0    60   Input ~ 0
-DXL_RXD_1
-Text GLabel 7200 3200 2    60   Input ~ 0
-DXL_485+_1
-Text GLabel 7200 3300 2    60   Input ~ 0
-DXL_485-_1
-Text GLabel 3550 4850 0    60   Input ~ 0
-DXL_485+_1
-Text GLabel 3550 4950 0    60   Input ~ 0
-DXL_485-_1
 $Comp
 L GND #PWR?
@@
 	1    0    0    -1
 $EndComp
-Text GLabel 3850 4450 1    60   Input ~ 0
-DXL_PWR
 $Comp
 L C C?
@@
 P 3850 5250
 F 0 "C?" H 3875 5350 50  0000 L CNN
-F 1 "C" H 3875 5150 50  0000 L CNN
+F 1 "0.1uF" H 3875 5150 50  0000 L CNN
 F 2 "" H 3888 5100 50  0001 C CNN
 F 3 "" H 3850 5250 50  0001 C CNN
@@
 	1    0    0    -1
 $EndComp
-Text GLabel 2900 8550 0    60   Input ~ 0
-DXL_PWR_EN
-$Comp
-L R R?
-U 1 1 5A69947A
-P 3700 7900
-F 0 "R?" V 3780 7900 50  0000 C CNN
-F 1 "R" V 3700 7900 50  0000 C CNN
-F 2 "" V 3630 7900 50  0001 C CNN
-F 3 "" H 3700 7900 50  0001 C CNN
-	1    3700 7900
-	1    0    0    -1
-$EndComp
-$Comp
-L C C?
-U 1 1 5A69952D
-P 4350 8550
-F 0 "C?" H 4375 8650 50  0000 L CNN
-F 1 "C" H 4375 8450 50  0000 L CNN
-F 2 "" H 4388 8400 50  0001 C CNN
-F 3 "" H 4350 8550 50  0001 C CNN
-	1    4350 8550
-	1    0    0    -1
-$EndComp
-Text GLabel 4950 9150 3    60   Input ~ 0
-DXL_PWR
-$Comp
-L R R?
-U 1 1 5A699733
-P 6650 8250
-F 0 "R?" V 6730 8250 50  0000 C CNN
-F 1 "R" V 6650 8250 50  0000 C CNN
-F 2 "" V 6580 8250 50  0001 C CNN
-F 3 "" H 6650 8250 50  0001 C CNN
-	1    6650 8250
-	1    0    0    -1
-$EndComp
-Text GLabel 4950 7250 1    60   Input ~ 0
-DC_BB_VCCIN
-$Comp
-L D_Schottky D?
-U 1 1 5A699A5F
-P 5550 8250
-F 0 "D?" H 5550 8350 50  0000 C CNN
-F 1 "D_Schottky" H 5550 8150 50  0000 C CNN
-F 2 "" H 5550 8250 50  0001 C CNN
-F 3 "" H 5550 8250 50  0001 C CNN
-	1    5550 8250
-	0    1    1    0
-$EndComp
-$Comp
-L D_Schottky D?
-U 1 1 5A699B12
-P 6100 8250
-F 0 "D?" H 6100 8350 50  0000 C CNN
-F 1 "D_Schottky" H 6100 8150 50  0000 C CNN
-F 2 "" H 6100 8250 50  0001 C CNN
-F 3 "" H 6100 8250 50  0001 C CNN
-	1    6100 8250
-	0    1    1    0
-$EndComp
-$Comp
-L C C?
-U 1 1 5A699B46
-P 6100 7800
-F 0 "C?" H 6125 7900 50  0000 L CNN
-F 1 "C" H 6125 7700 50  0000 L CNN
-F 2 "" H 6138 7650 50  0001 C CNN
-F 3 "" H 6100 7800 50  0001 C CNN
-	1    6100 7800
-	1    0    0    -1
-$EndComp
-$Comp
-L Q_PMOS_GDS Q?
-U 1 1 5A699B87
-P 4850 8200
-F 0 "Q?" H 5050 8250 50  0000 L CNN
-F 1 "Q_PMOS_GDS" H 5050 8150 50  0000 L CNN
-F 2 "" H 5050 8300 50  0001 C CNN
-F 3 "" H 4850 8200 50  0001 C CNN
-	1    4850 8200
-	1    0    0    1
-$EndComp
-$Comp
-L 2N2219 Q?
-U 1 1 5A69A90B
-P 3600 8550
-F 0 "Q?" H 3800 8625 50  0000 L CNN
-F 1 "2N2219" H 3800 8550 50  0000 L CNN
-F 2 "TO_SOT_Packages_THT:TO-39-3" H 3800 8475 50  0001 L CIN
-F 3 "" H 3600 8550 50  0001 L CNN
-	1    3600 8550
-	1    0    0    -1
-$EndComp
 Wire Wire Line
 	3550 3600 4300 3600
@@
 Wire Wire Line
 	4200 4650 4500 4650
-Wire Wire Line
-	4950 8400 4950 9150
-Wire Wire Line
-	4350 8950 6650 8950
-Wire Wire Line
-	4350 8950 4350 8700
-Wire Wire Line
-	6650 8950 6650 8400
-Connection ~ 4950 8950
-Wire Wire Line
-	3700 7750 3700 7450
-Wire Wire Line
-	3700 7450 6650 7450
-Wire Wire Line
-	6650 7450 6650 8100
-Wire Wire Line
-	4950 7250 4950 8000
-Connection ~ 4950 7450
-Wire Wire Line
-	4650 8200 3700 8200
-Wire Wire Line
-	4350 8400 4350 8200
-Connection ~ 4350 8200
-Wire Wire Line
-	5550 8100 5550 7450
-Connection ~ 5550 7450
-Wire Wire Line
-	6100 7650 6100 7450
-Connection ~ 6100 7450
-Wire Wire Line
-	6100 7950 6100 8100
-Wire Wire Line
-	6100 8400 6100 8950
-Connection ~ 6100 8950
-Wire Wire Line
-	5550 8400 5550 8950
-Connection ~ 5550 8950
-Wire Wire Line
-	3700 8050 3700 8350
-Connection ~ 3700 8200
-$Comp
-L GND #PWR?
-U 1 1 5A69AA92
-P 3700 9000
-F 0 "#PWR?" H 3700 8750 50  0001 C CNN
-F 1 "GND" H 3700 8850 50  0000 C CNN
-F 2 "" H 3700 9000 50  0001 C CNN
-F 3 "" H 3700 9000 50  0001 C CNN
-	1    3700 9000
-	1    0    0    -1
-$EndComp
-Wire Wire Line
-	3700 9000 3700 8750
-Wire Wire Line
-	3400 8550 2900 8550
 $Comp
 L MOLEX22-03-5045 J18?
@@
 	1    0    0    -1
 $EndComp
+$Comp
+L +5V #PWR?
+U 1 1 5A6FDCF8
+P 3750 2550
+F 0 "#PWR?" H 3750 2400 50  0001 C CNN
+F 1 "+5V" H 3750 2690 50  0000 C CNN
+F 2 "" H 3750 2550 50  0001 C CNN
+F 3 "" H 3750 2550 50  0001 C CNN
+	1    3750 2550
+	1    0    0    -1
+$EndComp
+Text HLabel 3550 3200 0    60   BiDi ~ 0
+DXL_RXD
+Text HLabel 3550 3500 0    60   BiDi ~ 0
+DXL_TXD
+Text HLabel 3550 3600 0    60   Input ~ 0
+DXL_DIR
+$Comp
+L +5V #PWR?
+U 1 1 5A6FED8C
+P 6100 3500
+F 0 "#PWR?" H 6100 3350 50  0001 C CNN
+F 1 "+5V" H 6100 3640 50  0000 C CNN
+F 2 "" H 6100 3500 50  0001 C CNN
+F 3 "" H 6100 3500 50  0001 C CNN
+	1    6100 3500
+	0    1    1    0
+$EndComp
+Text Label 7200 3200 0    60   ~ 0
+DXL_485+
+Text Label 7200 3300 0    60   ~ 0
+DXL_485-
+Text Label 3550 4850 2    60   ~ 0
+DXL_485+
+Text Label 3550 4950 2    60   ~ 0
+DXL_485-
+Text HLabel 3850 4450 0    60   Input ~ 0
+DXL_PWR
 $EndSCHEMATC
