File: NUsense/OTG-HS USB2o0.sch (KiCad schematic (older format))
At the start: 23 parts, among them J11? ZX62D-B-5P8, U16? EMIF02-USB03F2, U5? STMPS2141STR

Commit message: Change hierarchy layout
Parts:
- removed 0.1uF: C, symbol C
- removed R, R? (x2): R, symbol R
- removed U16?: EMIF02-USB03F2, symbol EMIF02-USB03F2
- removed U?: TUSB1210, symbol TUSB1210
- added C? (x4): C, symbol C
- added R?: R, symbol R
- added U?: USB3300-EZK, Housings_DFN_QFN:QFN-32-1EP_5x5mm_Pitch0.5mm, symbol USB3300-EZK
Connections:
- net labels added: +3.3V
- net labels removed: OTG_HS_PWR, VDD3o3V
- wire segments 66 -> 91

Commit message: Add power components
Parts:
- removed R? (x4): R, symbol R
- added C? (x9): C, symbol C
- added L?: Ferrite_Bead, symbol Ferrite_Bead
- added Q?: 2N3055, TO_SOT_Packages_THT:TO-3, symbol 2N3055
- added R? (x8): R, symbol R
- added U?: USBULC6-2F, symbol USBULC6-2F
- added U?: ESDA14V2-2BF3, symbol ESDA14V2-2BF3
- added Y?: Crystal, symbol Crystal
Connections:
- net labels added: +5V, EXTVBUS, OTG_HS_ULPI_CK, USB_EN
- net labels removed: VDD5o5V, VDD5o5V_USB
- wire segments 91 -> 129
Other:
- moved on the sheet: C?, D?, L?, R?, U?

Commit message: Update Component Values
Parts:
- removed C? (x6): C, symbol C
- added C? (x5): 100nF, symbol C
- added C?: 4.7uF, symbol C
- C: renamed from C?; value C -> 33pF
- C? (x2): value C -> 4.7uF
- C? (x5): value C -> 100nF
- Crystal: renamed from Y?; value Crystal -> 24MHz
- R: renamed from R?; value R -> 1M
- R: renamed from R?; value R -> 33
- R?: value R -> 10K
- R?: value R -> 3.3K
- R?: value R -> 620
- R? (x4): value R -> 0
- R?: value R -> 330
- R?: value R -> 820
- R?: value R -> 12K
- R?: value R -> 47K
- R?: value R -> 22K
Connections:
- net labels removed: USB_EN
Other:
- moved on the sheet: C?

Commit message: ESD protection
Parts:
- removed U?: USBULC6-2F, symbol USBULC6-2F
- removed U?: ESDA14V2-2BF3, symbol ESDA14V2-2BF3
- added C?: 10Uf, symbol C
- added R?: 10K, symbol R
- added U?: TPD4S014, symbol TPD4S014
Connections:
- net labels added: USB_~ACK
- wire segments 129 -> 139
Changed lines of the file:
@@
 	8650 3750 8950 3750
-Wire Wire Line
-	9250 3750 11600 3750
 Wire Wire Line
 	8800 3750 8800 3250
@@
 Connection ~ 11550 2500
 $Comp
-L USBULC6-2F U?
-U 1 1 5A714118
-P 9950 4750
-F 0 "U?" H 10300 4950 60  0000 C CNN
-F 1 "USBULC6-2F" H 10550 4800 60  0000 C CNN
-F 2 "" H 9950 4750 60  0001 C CNN
-F 3 "" H 9950 4750 60  0001 C CNN
-	1    9950 4750
-	1    0    0    -1
-$EndComp
-$Comp
-L ESDA14V2-2BF3 U?
-U 1 1 5A714187
-P 11050 4750
-F 0 "U?" H 11400 4950 60  0000 C CNN
-F 1 "ESDA14V2-2BF3" H 11750 4800 60  0000 C CNN
-F 2 "" H 11050 4750 60  0001 C CNN
-F 3 "" H 11050 4750 60  0001 C CNN
-	1    11050 4750
-	1    0    0    -1
-$EndComp
-$Comp
-L GND #PWR?
-U 1 1 5A714880
-P 10150 5050
-F 0 "#PWR?" H 10150 4800 50  0001 C CNN
-F 1 "GND" H 10150 4900 50  0000 C CNN
-F 2 "" H 10150 5050 50  0001 C CNN
-F 3 "" H 10150 5050 50  0001 C CNN
-	1    10150 5050
-	1    0    0    -1
-$EndComp
-$Comp
-L GND #PWR?
-U 1 1 5A7148FD
-P 11250 5050
-F 0 "#PWR?" H 11250 4800 50  0001 C CNN
-F 1 "GND" H 11250 4900 50  0000 C CNN
-F 2 "" H 11250 5050 50  0001 C CNN
-F 3 "" H 11250 5050 50  0001 C CNN
-	1    11250 5050
-	1    0    0    -1
-$EndComp
-Wire Wire Line
-	11250 4950 11250 5050
-Wire Wire Line
-	11150 4950 11150 5000
-Wire Wire Line
-	11150 5000 11250 5000
-Connection ~ 11250 5000
-Wire Wire Line
-	10050 4950 10050 5000
-Wire Wire Line
-	10050 5000 10150 5000
-Wire Wire Line
-	10150 4950 10150 5050
-Connection ~ 10150 5000
-Wire Wire Line
-	10050 3950 10050 4200
-Connection ~ 10050 3950
-Wire Wire Line
-	10150 3850 10150 4200
-Connection ~ 10150 3850
-Wire Wire Line
-	11150 4200 11150 4050
-Connection ~ 11150 4050
-Wire Wire Line
-	11250 4200 11250 3750
-Connection ~ 11250 3750
-$Comp
 L C C?
 U 1 1 5A715539
@@
 	5150 4100 5050 4100
 Wire Wire Line
-	11400 3750 11400 3500
+	11400 3500 11400 4500
 Wire Wire Line
 	11400 3500 11950 3500
 Wire Wire Line
 	11950 3500 11950 3350
-Connection ~ 11400 3750
 $Comp
 L +5V #PWR?
@@
 	13550 4900 13550 4800
 Connection ~ 13550 4800
+$Comp
+L TPD4S014 U?
+U 1 1 5A72B380
+P 10300 4900
+F 0 "U?" H 10700 5550 60  0000 C CNN
+F 1 "TPD4S014" H 10650 4850 60  0000 C CNN
+F 2 "" H 10300 4900 60  0001 C CNN
+F 3 "" H 10300 4900 60  0001 C CNN
+	1    10300 4900
+	1    0    0    -1
+$EndComp
+Wire Wire Line
+	11150 4700 11600 4700
+Wire Wire Line
+	11600 4700 11600 3950
+Connection ~ 11600 3950
+Wire Wire Line
+	11150 4800 11700 4800
+Wire Wire Line
+	11700 4800 11700 3850
+Connection ~ 11700 3850
+Wire Wire Line
+	10100 4800 9650 4800
+Wire Wire Line
+	9650 4800 9650 4050
+Connection ~ 9650 4050
+Wire Wire Line
+	11400 4400 11150 4400
+Wire Wire Line
+	11400 4500 11150 4500
+Connection ~ 11400 4400
+Wire Wire Line
+	11400 4150 11900 4150
+Wire Wire Line
+	11900 4150 11900 4250
+Connection ~ 11400 4150
+$Comp
+L C C?
+U 1 1 5A72C99B
+P 11900 4400
+F 0 "C?" H 11925 4500 50  0000 L CNN
+F 1 "10Uf" H 11925 4300 50  0000 L CNN
+F 2 "" H 11938 4250 50  0001 C CNN
+F 3 "" H 11900 4400 50  0001 C CNN
+	1    11900 4400
+	1    0    0    -1
+$EndComp
+$Comp
+L GND #PWR?
+U 1 1 5A72CA08
+P 11900 4700
+F 0 "#PWR?" H 11900 4450 50  0001 C CNN
+F 1 "GND" H 11900 4550 50  0000 C CNN
+F 2 "" H 11900 4700 50  0001 C CNN
+F 3 "" H 11900 4700 50  0001 C CNN
+	1    11900 4700
+	1    0    0    -1
+$EndComp
+Wire Wire Line
+	11900 4700 11900 4550
+Wire Wire Line
+	11150 4600 11900 4600
+Connection ~ 11900 4600
+Wire Wire Line
+	11400 3750 11600 3750
+Connection ~ 11400 3750
+Wire Wire Line
+	10100 4400 10000 4400
+Wire Wire Line
+	10000 3750 10000 4500
+Wire Wire Line
+	10000 4500 10100 4500
+Wire Wire Line
+	10000 3750 9250 3750
+Connection ~ 10000 4400
+Wire Wire Line
+	10100 4600 9900 4600
+Wire Wire Line
+	9900 4600 9900 5050
+$Comp
+L GND #PWR?
+U 1 1 5A72D25B
+P 9900 5050
+F 0 "#PWR?" H 9900 4800 50  0001 C CNN
+F 1 "GND" H 9900 4900 50  0000 C CNN
+F 2 "" H 9900 5050 50  0001 C CNN
+F 3 "" H 9900 5050 50  0001 C CNN
+	1    9900 5050
+	1    0    0    -1
+$EndComp
+Text HLabel 8950 4700 0    60   Input ~ 0
+USB_~ACK
+Wire Wire Line
+	10100 4700 8950 4700
+$Comp
+L R R?
+U 1 1 5A72DCA1
+P 9200 4500
+F 0 "R?" V 9280 4500 50  0000 C CNN
+F 1 "10K" V 9200 4500 50  0000 C CNN
+F 2 "" V 9130 4500 50  0001 C CNN
+F 3 "" H 9200 4500 50  0001 C CNN
+	1    9200 4500
+	-1   0    0    1
+$EndComp
+$Comp
+L +3.3V #PWR?
+U 1 1 5A72DDFF
+P 9200 4350
+F 0 "#PWR?" H 9200 4200 50  0001 C CNN
+F 1 "+3.3V" H 9200 4490 50  0000 C CNN
+F 2 "" H 9200 4350 50  0001 C CNN
+F 3 "" H 9200 4350 50  0001 C CNN
+	1    9200 4350
+	1    0    0    -1
+$EndComp
+Wire Wire Line
+	9200 4650 9200 4700
+Connection ~ 9200 4700
 $EndSCHEMATC

Commit message: Adds annotations and footprints to all components
Parts:
- C701, C702: renamed from C; value 33pF -> 10pF; footprint (none) -> Capacitors_SMD:C_0805_HandSoldering
- C703, C704, C705, C706, C707, C708, C709, C710, C711, C712, C713, C714, C715, C716: renamed from C?; footprint (none) -> Capacitors_SMD:C_0805_HandSoldering
- Q701: renamed from Q?; footprint TO_SOT_Packages_THT:TO-3 -> TO_SOT_Packages_SMD:SOT-23
- R701, R706: renamed from R; footprint (none) -> Resistors_SMD:R_0805_HandSoldering
- R702, R703, R704, R705, R707, R708, R709, R710, R711, R712, R713, R714, R715: renamed from R?; footprint (none) -> Resistors_SMD:R_0805_HandSoldering
- U5701: renamed from U5?; footprint (none) -> TO_SOT_Packages_SMD:SOT-23-5_HandSoldering
- U701: renamed from U?; footprint Housings_DFN_QFN:QFN-32-1EP_5x5mm_Pitch0.5mm -> Footprints:QFP_32_T
- X701: renamed from Crystal; footprint (none) -> Footprints:XTAL-OSC; symbol Crystal -> Crystal_GND24
- gave numbers to parts that had none: 7
Connections:
- net GND: now also X701.2, X701.4
- net at C702.1, R701.1, U701.28 (XI): now also X701.3; no longer X701.2
Other:
- moved on the sheet: C701, C702

Commit message: More Changes
Parts:
- removed F701: Fuse, symbol Fuse
- renumbered C701 to C601, C702 to C602, C703 to C603, C704 to C604, C705 to C605, C706 to C606, C707 to C607, C708 to C608, C709 to C609, C710 to C610, C711 to C611, C712 to C612, C713 to C613, C714 to C614, C715 to C615, C716 to C616, D701 to D601, D702 to D602, J11701 to J601, L701 to L601, L702 to L602, Q701 to Q601, R701 to R601, R702 to R602, R703 to R603, R704 to R604, R705 to R605, R706 to R606, R707 to R607, R708 to R608, R709 to R609, R710 to R610, R711 to R611, R712 to R612, R713 to R613, R714 to R614, R715 to R615, U701 to U601, U5701 to U602, U702 to U603, X701 to X601
Connections:
- net +5V: now also J601.1 (VBUS)
