File: NUsense/Voltage_Sensor.sch (KiCad schematic (older format))
At the start: 24 parts, among them U701 ACS724, U702 bq76920, U703 5_PIN_JST

Commit message: Further Changes
Parts:
- C701, C703, C706, C707, C708, C709, C710: value C -> 1uF
- C702: value C -> 4.7uF
- C704: value C -> 10uF
- R701: value R_Variable -> 10K
- R702: value R -> 10K
- R703, R705, R706, R707, R708, R709: value R -> 100
Changed lines of the file:
@@
 P 5100 4350
 F 0 "R707" V 5180 4350 50  0000 C CNN
-F 1 "R" V 5100 4350 50  0000 C CNN
+F 1 "100" V 5100 4350 50  0000 C CNN
 F 2 "Resistors_SMD:R_0805_HandSoldering" V 5030 4350 50  0001 C CNN
 F 3 "" H 5100 4350 50  0001 C CNN
@@
 P 5100 3150
 F 0 "R705" V 5180 3150 50  0000 C CNN
-F 1 "R" V 5100 3150 50  0000 C CNN
+F 1 "100" V 5100 3150 50  0000 C CNN
 F 2 "Resistors_SMD:R_0805_HandSoldering" V 5030 3150 50  0001 C CNN
 F 3 "" H 5100 3150 50  0001 C CNN
@@
 P 5100 3950
 F 0 "R706" V 5180 3950 50  0000 C CNN
-F 1 "R" V 5100 3950 50  0000 C CNN
+F 1 "100" V 5100 3950 50  0000 C CNN
 F 2 "Resistors_SMD:R_0805_HandSoldering" V 5030 3950 50  0001 C CNN
 F 3 "" H 5100 3950 50  0001 C CNN
@@
 P 4800 3750
 F 0 "C707" H 4825 3850 50  0000 L CNN
-F 1 "C" H 4825 3650 50  0000 L CNN
+F 1 "1uF" H 4825 3650 50  0000 L CNN
 F 2 "Capacitors_SMD:C_0805_HandSoldering" H 4838 3600 50  0001 C CNN
 F 3 "" H 4800 3750 50  0001 C CNN
@@
 P 4800 4150
 F 0 "C708" H 4825 4250 50  0000 L CNN
-F 1 "C" H 4825 4050 50  0000 L CNN
+F 1 "1uF" H 4825 4050 50  0000 L CNN
 F 2 "Capacitors_SMD:C_0805_HandSoldering" H 4838 4000 50  0001 C CNN
 F 3 "" H 4800 4150 50  0001 C CNN
@@
 P 5100 4750
 F 0 "R708" V 5180 4750 50  0000 C CNN
-F 1 "R" V 5100 4750 50  0000 C CNN
+F 1 "100" V 5100 4750 50  0000 C CNN
 F 2 "Resistors_SMD:R_0805_HandSoldering" V 5030 4750 50  0001 C CNN
 F 3 "" H 5100 4750 50  0001 C CNN
@@
 P 4800 4550
 F 0 "C709" H 4825 4650 50  0000 L CNN
-F 1 "C" H 4825 4450 50  0000 L CNN
+F 1 "1uF" H 4825 4450 50  0000 L CNN
 F 2 "Capacitors_SMD:C_0805_HandSoldering" H 4838 4400 50  0001 C CNN
 F 3 "" H 4800 4550 50  0001 C CNN
@@
 P 5100 5150
 F 0 "R709" V 5180 5150 50  0000 C CNN
-F 1 "R" V 5100 5150 50  0000 C CNN
+F 1 "100" V 5100 5150 50  0000 C CNN
 F 2 "Resistors_SMD:R_0805_HandSoldering" V 5030 5150 50  0001 C CNN
 F 3 "" H 5100 5150 50  0001 C CNN
@@
 P 4800 4950
 F 0 "C710" H 4825 5050 50  0000 L CNN
-F 1 "C" H 4825 4850 50  0000 L CNN
+F 1 "1uF" H 4825 4850 50  0000 L CNN
 F 2 "Capacitors_SMD:C_0805_HandSoldering" H 4838 4800 50  0001 C CNN
 F 3 "" H 4800 4950 50  0001 C CNN
@@
 P 4800 3350
 F 0 "C706" H 4825 3450 50  0000 L CNN
-F 1 "C" H 4825 3250 50  0000 L CNN
+F 1 "1uF" H 4825 3250 50  0000 L CNN
 F 2 "Capacitors_SMD:C_0805_HandSoldering" H 4838 3200 50  0001 C CNN
 F 3 "" H 4800 3350 50  0001 C CNN
@@
 P 2300 4300
 F 0 "R702" V 2380 4300 50  0000 C CNN
-F 1 "R" V 2300 4300 50  0000 C CNN
+F 1 "10K" V 2300 4300 50  0000 C CNN
 F 2 "Resistors_SMD:R_0805_HandSoldering" V 2230 4300 50  0001 C CNN
 F 3 "" H 2300 4300 50  0001 C CNN
@@
 P 1950 3950
 F 0 "R701" V 2050 3850 50  0000 L CNN
-F 1 "R_Variable" V 1850 3900 50  0000 L CNN
+F 1 "10K" V 1850 3900 50  0000 L CNN
 F 2 "Resistors_SMD:R_0805_HandSoldering" V 1880 3950 50  0001 C CNN
 F 3 "" H 1950 3950 50  0001 C CNN
@@
 P 2450 5400
 F 0 "C702" H 2475 5500 50  0000 L CNN
-F 1 "C" H 2475 5300 50  0000 L CNN
+F 1 "4.7uF" H 2475 5300 50  0000 L CNN
 F 2 "Capacitors_SMD:C_0805_HandSoldering" H 2488 5250 50  0001 C CNN
 F 3 "" H 2450 5400 50  0001 C CNN
@@
 	2450 5550 2450 5650
 Wire Wire Line
-	2450 5150 2200 5150
-Wire Wire Line
-	2200 5150 2200 5600
+	1850 5150 2450 5150
 Connection ~ 2450 5150
 $Comp
@@
 P 2700 4850
 F 0 "R703" V 2780 4850 50  0000 C CNN
-F 1 "R" V 2700 4850 50  0000 C CNN
+F 1 "100" V 2700 4850 50  0000 C CNN
 F 2 "Resistors_SMD:R_0805_HandSoldering" V 2630 4850 50  0001 C CNN
 F 3 "" H 2700 4850 50  0001 C CNN
@@
 P 2950 4800
 F 0 "C704" H 2975 4900 50  0000 L CNN
-F 1 "C" H 2975 4700 50  0000 L CNN
+F 1 "10uF" H 2975 4700 50  0000 L CNN
 F 2 "Capacitors_SMD:C_0805_HandSoldering" H 2988 4650 50  0001 C CNN
 F 3 "" H 2950 4800 50  0001 C CNN
 	1    2950 4800
-	-1   0    0    -1
+	1    0    0    -1
 $EndComp
 Wire Wire Line
@@
 P 2150 4800
 F 0 "C701" H 2175 4900 50  0000 L CNN
-F 1 "C" H 2175 4700 50  0000 L CNN
+F 1 "1uF" H 2175 4700 50  0000 L CNN
 F 2 "Capacitors_SMD:C_0805_HandSoldering" H 2188 4650 50  0001 C CNN
 F 3 "" H 2150 4800 50  0001 C CNN
@@
 P 2700 5300
 F 0 "C703" H 2725 5400 50  0000 L CNN
-F 1 "C" H 2725 5200 50  0000 L CNN
+F 1 "1uF" H 2725 5200 50  0000 L CNN
 F 2 "Capacitors_SMD:C_0805_HandSoldering" H 2738 5150 50  0001 C CNN
 F 3 "" H 2700 5300 50  0001 C CNN
@@
 L +3.3V #PWR076
 U 1 1 5A719D8E
-P 2200 5600
-F 0 "#PWR076" H 2200 5450 50  0001 C CNN
-F 1 "+3.3V" H 2200 5740 50  0000 C CNN
-F 2 "" H 2200 5600 50  0001 C CNN
-F 3 "" H 2200 5600 50  0001 C CNN
-	1    2200 5600
-	-1   0    0    1
+P 1850 5100
+F 0 "#PWR076" H 1850 4950 50  0001 C CNN
+F 1 "+3.3V" H 1850 5240 50  0000 C CNN
+F 2 "" H 1850 5100 50  0001 C CNN
+F 3 "" H 1850 5100 50  0001 C CNN
+	1    1850 5100
+	1    0    0    -1
 $EndComp
 Wire Wire Line
@@
 Text HLabel 1600 1800 0    60   BiDi ~ 0
 BATT_-
+Wire Wire Line
+	1850 5100 1850 5150
 $EndSCHEMATC
