Commit message: Update upper body
Still need to fix up more
- Add correct physics
- Add better mesh models
- Better position visual mesh's

File: Models/URDF/urdf/NUgus.urdf (robot description, URDF)
Before this commit: robot nubots_nugus_hull, 21 links, 20 joints
Joints:
- joint head_pitch: axis 1  0  0 -> 0 0 1; origin xyz=0  0  0 rpy=0  0  0 -> xyz=0  0  0 rpy=1.571  0  0
- joint left_elbow_pitch: origin xyz=-0.01    -0.19     0.03999 rpy=0  0  0 -> xyz=0.1575 -0.005 0 rpy=-1.571  0  0
- joint left_shoulder_pitch: origin xyz=0.005  0.115  0.18 rpy=-1.571 0 0 -> xyz=0 0.077 0.17725 rpy=-1.571 0 0
- joint left_shoulder_roll: origin xyz=0.015  0     0.005 rpy=0 0 1 -> xyz=0.01 0 0.047 rpy=1.571 0 0
- joint neck_yaw: origin xyz=0    0    0.26 rpy=0       0       1.57079 -> xyz=0 0 0.26 rpy=0 0 0
- joint right_elbow_pitch: origin xyz=0.01 -0.19  0.04 rpy=0  0  0 -> xyz=0.1575 0 0 rpy=-1.571  0  0
- joint right_shoulder_pitch: origin xyz=0.005 -0.115  0.18 rpy=-1.571 0 0 -> xyz=0 -0.077 0.17725 rpy=-1.571 0 0
- joint right_shoulder_roll: origin xyz=-0.015  0     0.005 rpy=0 0 1 -> xyz=0.01 0 -0.047 rpy=1.571 0 0
