File: NU740/nu740_board/power.kicad_sch (KiCad schematic)
At the start: 23 parts, among them J12 Conn_01x02, Q2 SUD50P06-15, Q3 MMBT3904, U1 TPS54302, U6 L78L33_SOT89

Commit message: Too long ago to remember.
Parts:
- added C31: 22μ, Capacitor_SMD:C_0805_2012Metric, symbol Device:C
- C1: value C -> 10μ; footprint (none) -> Capacitor_SMD:C_0805_2012Metric
- C2, C4: value C -> 100n; footprint (none) -> Capacitor_SMD:C_0603_1608Metric
- C3: value C -> 22μ; footprint (none) -> Capacitor_SMD:C_0805_2012Metric
- L1: value L -> 10μ; footprint (none) -> Inductor_SMD:L_Neosid_Ms42
- R1: value R_US -> 100k; footprint (none) -> Resistor_SMD:R_0603_1608Metric
- R2: value R_US -> 13.3k; footprint (none) -> Resistor_SMD:R_0603_1608Metric
Connections:
- net +5V: now also C31.1
- net GND: now also C31.2
Other:
- moved on the sheet: R21
