File: NU740/nu740_board/usb.kicad_sch (KiCad schematic)
At the start: 34 parts, among them J11 USB_C_Receptacle_USB2.0_16P, J3 USB_B_Micro, J4 Conn_01x04, Q1 IRLML6402, U4 SP485EEN, U5 FT232RNL

Commit message: Too long ago to remember.
Connections:
- no-connect marks 10 -> 11
